File: ADR1399E_ref_board.kicad_sch (KiCad schematic)
At the start: 32 parts, among them J1 USB_C_Receptacle_PowerOnly_6P, J2 Conn_01x02_Pin, U1 ADR1399KEZ, U2 LT3042xMSE, U3 TPS61085DGK, U4 TL331, U5 OPA182IDR

Commit message: moving forward
Parts:
- removed C6: 100n 50V, Capacitor_SMD:C_0504_1310Metric_Pad0.83x1.28mm_HandSolder, symbol Device:C
- removed C8: 10uF 50V, Capacitor_SMD:C_1210_3225Metric_Pad1.33x2.70mm_HandSolder, symbol Device:C
- added C1, C2, C3: 10uF 10V, Capacitor_SMD:C_0805_2012Metric_Pad1.18x1.45mm_HandSolder, symbol Device:C
- added C10: 10uF 50V, nightmechanic_pcb:3225_Kelvin_4port, symbol nightmechanic_lib:Kelvin_Cap
- added C12: 10uF 50V, Capacitor_SMD:C_1210_3225Metric_Pad1.33x2.70mm_HandSolder, symbol Device:C
- added C14, C15: 100n 50V, Capacitor_SMD:C_0603_1608Metric_Pad1.08x0.95mm_HandSolder, symbol Device:C
- added C16: 1uF 25V, Capacitor_SMD:C_0603_1608Metric_Pad1.08x0.95mm_HandSolder, symbol Device:C
- added C4: 330n 50V, Capacitor_SMD:C_0603_1608Metric_Pad1.08x0.95mm_HandSolder, symbol Device:C
- added D1: LED, LED_SMD:LED_1206_3216Metric_Pad1.42x1.75mm_HandSolder, symbol Device:LED
- added J3: Conn_Coaxial, Connector_Coaxial:SMA_Molex_73251-1153_EdgeMount_Horizontal, symbol Connector:Conn_Coaxial
- added R13, R14: 1.5k, Resistor_SMD:R_0805_2012Metric_Pad1.20x1.40mm_HandSolder, symbol Device:R
- added R17: 20k, Resistor_SMD:R_0805_2012Metric_Pad1.20x1.40mm_HandSolder, symbol Device:R
- added R18: 8.37k, Resistor_SMD:R_0805_2012Metric_Pad1.20x1.40mm_HandSolder, symbol Device:R
- added R19: 5R, Resistor_SMD:R_0805_2012Metric_Pad1.20x1.40mm_HandSolder, symbol Device:R
- added R3: 366k, Resistor_SMD:R_0805_2012Metric_Pad1.20x1.40mm_HandSolder, symbol Device:R
- added R5: 5.1k, Resistor_SMD:R_0805_2012Metric_Pad1.20x1.40mm_HandSolder, symbol Device:R
- added R8: 10k, Resistor_SMD:R_0805_2012Metric_Pad1.20x1.40mm_HandSolder, symbol Device:R
- added TP1: TestPoint, TestPoint:TestPoint_Pad_D1.5mm, symbol Connector:TestPoint
- C11: renamed from C5; footprint Capacitor_SMD:C_0504_1310Metric_Pad0.83x1.28mm_HandSolder -> Capacitor_SMD:C_0603_1608Metric_Pad1.08x0.95mm_HandSolder
- C13: renamed from C4; footprint Capacitor_SMD:C_0504_1310Metric_Pad0.83x1.28mm_HandSolder -> Capacitor_SMD:C_0603_1608Metric_Pad1.08x0.95mm_HandSolder
- C7: value 4.7uF 50V -> 330n 50V; footprint Capacitor_SMD:C_1206_3216Metric_Pad1.33x1.80mm_HandSolder -> Capacitor_SMD:C_0603_1608Metric_Pad1.08x0.95mm_HandSolder
- renumbered C2 to C5, C1 to C6, C3 to C8, J2 to J1, J1 to J2, R2 to R1, R4 to R10, R5 to R11, R3 to R12, R6 to R15, R1 to R16, R8 to R2, R10 to R4, R9 to R6, R12 to R9, U2 to U1, U3 to U2, U4 to U3, U5 to U4, U1 to U5
Connections:
- net at R15.1: now also R11.2, U3.1 (-)
- net GND: now reaches R15.2
- net GND: now also C11.2, C13.2, C5.2, C6.2, C7.2, C8.2, C9.2, J1.1 (Pin_1), J2.A12 (GND), J2.B12 (GND), J2.S1 (SHIELD), R16.2, R4.2, R6.2, U1.11 (GND), U1.5 (ILIM), U1.8 (GND), U2.4 (GND), U2.7 (FREQ), U3.2 (V-), U4.4 (V-), U5.1 (-REFS), U5.2 (-REFF), U5.5 (HEATER-), C1.2, C10.2, C14.2, C15.2, C2.2, C3.2, C4.2, D1.1 (K), J3.2 (Ext), R17.2, R19.2, R5.2, R8.2
- net +12V: now reaches U5.3 (HEATER+)
- net +12V: now also U1.10 (OUT), U4.7 (V+), C10.3, C14.1, C15.1, R13.1, R14.1, R3.1
- net at U5.6 (+REFF): now also U4.3 (+IN), U5.7 (+REFS), C16.1, R14.2
- net +BATT: now reaches R11.1
- net +BATT: now also CR1.1, J1.2 (Pin_2)
- net at R7.1: now also U2.1 (COMP)
- net at R7.2: now also C13.1
- net Inductance: now reaches CR1.2
- net Inductance: now also C7.1, C8.1, C9.1, L2.2, U1.1 (IN), U1.2 (IN), U1.3 (EN/UV)
- net at U2.2 (FB): now also R2.2, R6.1
- net Boost_En: now reaches U2.3 (EN)
- net Boost_En: now also R1.2, R10.2, U3.4
- net at U2.5 (SW): now also CR2.1, L1.2
- net +5V: now reaches U2.6 (VIN)
- net +5V: now also J2.A9 (VBUS), J2.B9 (VBUS), L1.1, R1.1, R12.1, U3.5 (V+), C1.1, C2.1, C3.1
- net at U2.8 (SS): now also C11.1
- net at C6.1: now also C5.1, CR2.2, CR3.1, R2.1, C4.1
- net at R4.1: now also J2.A5 (CC1)
- net at J2.B5 (CC2): now also R5.1
- net at U1.4 (PG): now also TP1.1
- net at U1.6 (PGFB): now also R3.2, R8.1
- net at U1.7 (SET): now also R9.1, C12.1
- net at U1.9 (OUTS): now also C10.4
- net at R12.2: now also R10.1, R16.1, U3.3 (+)
- net at L2.1: now also CR3.2
- net at R9.2: now also C10.1, C12.2
- net at U4.2 (-IN): now also R17.1, R18.1
- net at U4.6 (OUT): now also J3.1 (In), R18.2
- new net: D1.2 (A), R13.2
- new net: C16.2, R19.1
Other:
- note added: "PCB inductance: 2mm wide 15mm long"
- moved on the sheet: C11, C13, C5, C6, C8, C9, CR1, CR2, CR3, J1, L1, L2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

Commit message: getting closer
Parts:
- removed R18: 8.37k, Resistor_SMD:R_0805_2012Metric_Pad1.20x1.40mm_HandSolder, symbol Device:R
- removed U4: OPA182IDR, Snapeda:D0008A-IPC_A, symbol Snapeda:OPA182IDR
- added C17: 1uF 25V, Capacitor_SMD:C_0603_1608Metric_Pad1.08x0.95mm_HandSolder, symbol Device:C
- added IC1: OPA189IDR, Samacsys:SOIC127P600X175-8N, symbol Samacsys:OPA189IDR
- added JP1, JP10, JP11, JP13, JP2, JP3, JP4, JP5, JP6, JP7, JP8, JP9: SolderJumper_2_Open, Jumper:SolderJumper-2_P1.3mm_Open_RoundedPad1.0x1.5mm, symbol Jumper:SolderJumper_2_Open
- added RN1: R_Pack08, Package_SO:SO-16_3.9x9.9mm_P1.27mm, symbol Device:R_Pack08
- R14: value 1.5k -> 200k
- R17: value 20k -> 4R7
Connections:
- net +12V: now also C17.1, IC1.7 (V+)
- net GND: now also C17.2, IC1.4 (V-), JP3.2 (B), JP7.2 (B), JP8.2 (B), JP9.2 (B); no longer R17.2
- net at C16.1, R14.2, U5.6 (+REFF)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: now also IC1.3 (+IN), RN1.1 (R1.1)
- net at J3.1 (In): now also R17.1, IC1.6 (OUT), RN1.16 (R1.2)
- new net: JP1.1 (A), JP10.2 (B), JP11.2 (B), JP3.1 (A), RN1.12 (R5.2)
- new net: JP1.2 (B), JP7.1 (A), RN1.11 (R6.2)
- new net: JP8.1 (A), RN1.10 (R7.2)
- new net: RN1.13 (R4.2), RN1.14 (R3.2)
- new net: R17.2, RN1.15 (R2.2)
- new net: IC1.2 (-IN), RN1.2 (R2.1), RN1.3 (R3.1)
- new net: JP10.1 (A), JP13.2 (B), JP2.2 (B), RN1.4 (R4.1)
- new net: JP2.1 (A), JP4.2 (B), RN1.5 (R5.1)
- new net: JP4.1 (A), JP5.2 (B), RN1.6 (R6.1)
- new net: JP11.1 (A), JP5.1 (A), JP6.2 (B), RN1.7 (R7.1)
- new net: JP13.1 (A), JP6.1 (A), RN1.8 (R8.1)
- new net: JP9.1 (A), RN1.9 (R8.2)
- no-connect marks 0 -> 3
Other:
- note added: "Ref Zener Bias"
- company: (none) -> Nightmechanics
- title: (none) -> ADR1399 refernce board
- moved on the sheet: C14, C15, C16, D1, J3, R13, R14, R19, U5

Commit message: complete schematics?
Parts:
- added P1: JST_B2P_VH, Connector_JST:JST_VH_B2P-VH_1x02_P3.96mm_Vertical, symbol nightmechanic_lib:JST_B2PS_VH
- added TP1, TP2, TP3, TP4, TP6, TP7, TP8, TP9: TestPoint, TestPoint:TestPoint_Loop_D1.80mm_Drill1.0mm_Beaded, symbol Connector:TestPoint
- renumbered C17 to C15, C15 to C16, C16 to C17, JP2 to JP1, JP13 to JP10, JP10 to JP11, JP11 to JP12, JP3 to JP2, JP1 to JP3, JP7 to JP6, JP6 to JP7, R13 to R11, R14 to R12, R11 to R13, R12 to R14, R17 to R15, R15 to R16, R16 to R17, R19 to R18, TP1 to TP5, U5 to U4
Connections:
- net +12V: now also TP4.1
- net +5V: now also TP2.1
- net GND: now also P1.2, TP6.1, TP9.1
- net Inductance: now also TP1.1
- net at C17.1, IC1.3 (+IN), R12.2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: now also TP7.1
- net at IC1.6 (OUT), J3.1 (In), R15.1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: now also P1.1, TP8.1
- net at C4.1, C5.1, C6.1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: now also TP3.1

Commit message: buffered output, temp sensor, resistor network
Parts:
- removed IC1: OPA189IDR, Samacsys:SOIC127P600X175-8N, symbol Samacsys:OPA189IDR
- added C19, C23: 1uF 25V, Capacitor_SMD:C_0603_1608Metric_Pad1.08x0.95mm_HandSolder, symbol Device:C
- added C20: 1n 25V, Capacitor_SMD:C_0603_1608Metric_Pad1.08x0.95mm_HandSolder, symbol Device:C
- added C21: 3n 25V, Capacitor_SMD:C_0603_1608Metric_Pad1.08x0.95mm_HandSolder, symbol Device:C
- added C24: 100n 50V, Capacitor_SMD:C_0603_1608Metric_Pad1.08x0.95mm_HandSolder, symbol Device:C
- added D2: PTVS11VP1UP,115, Samacsys:PMEG3050EP115, symbol Samacsys:PTVS11VP1UP,115
- added J4: S4B-XH-A, Connector_JST:JST_XH_S4B-XH-A_1x04_P2.50mm_Horizontal, symbol Connector:Conn_01x04_Socket
- added Q1: MMBT3906, Package_TO_SOT_SMD:SOT-23, symbol Transistor_BJT:MMBT3906
- added R19: 0R, Resistor_SMD:R_0805_2012Metric_Pad1.20x1.40mm_HandSolder, symbol Device:R
- added R20: 10R, Resistor_SMD:R_0805_2012Metric_Pad1.20x1.40mm_HandSolder, symbol Device:R
- added R22: 1R, Resistor_SMD:R_0805_2012Metric_Pad1.20x1.40mm_HandSolder, symbol Device:R
- added R23: 1k 0.1% 5ppm, Resistor_SMD:R_0603_1608Metric_Pad0.98x0.95mm_HandSolder, symbol Device:R
- added R24: 10k 0.1% 10ppm, Resistor_SMD:R_0805_2012Metric_Pad1.20x1.40mm_HandSolder, symbol Device:R
- added R25: 7.5k, Resistor_SMD:R_0805_2012Metric_Pad1.20x1.40mm_HandSolder, symbol Device:R
- added R26: 100k, Resistor_SMD:R_0805_2012Metric_Pad1.20x1.40mm_HandSolder, symbol Device:R
- added U5: LMT01LPG, Package_TO_SOT_THT:TO-92-2, symbol Sensor_Temperature:LMT01LPG
- added U6: OPA182IDR, Snapeda:D0008A-IPC_A, symbol Snapeda:OPA182IDR
- added U7: OPA994IDR, Snapeda:D0008A-IPC_A, symbol Snapeda:OPA182IDR
- R15: value 4R7 -> 0R
- RN1: value R_Pack08 -> 10k x8
Connections:
- net +12V: now also R19.1; no longer C14.1, C15.1, C16.1, R11.1, R12.1, U4.3 (HEATER+)
- net GND: now also C19.2, C23.2, C24.2, D2.2 (A), R24.2, U6.4 (V-), U7.4 (V-)
- net at C17.1, R12.2, TP7.1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: now also R23.1, U6.3 (+IN); no longer RN1.1 (R1.1)
- net at JP11.2 (B), JP12.2 (B), JP2.1 (A)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: now also RN1.13 (R4.2); no longer RN1.12 (R5.2)
- net at JP3.2 (B), JP6.1 (A): now also RN1.12 (R5.2); no longer RN1.11 (R6.2)
- net at JP8.1 (A): now also RN1.11 (R6.2); no longer RN1.10 (R7.2)
- net at RN1.14 (R3.2): now also RN1.15 (R2.2); no longer RN1.13 (R4.2)
- net 10V_Out: now reaches R15.2
- net 10V_Out: now also J3.1 (In), P1.1, TP8.1, D2.1 (K), R22.2, R23.2, R24.1; no longer RN1.15 (R2.2)
- net at RN1.2 (R2.1): now also RN1.1 (R1.1), C20.1, C21.1, U6.2 (-IN); no longer RN1.3 (R3.1)
- net at JP1.2 (B), JP10.2 (B), JP11.1 (A): now also RN1.3 (R3.1); no longer RN1.4 (R4.1)
- net at JP1.1 (A), JP4.2 (B): now also RN1.4 (R4.1); no longer RN1.5 (R5.1)
- net at JP4.1 (A), JP5.2 (B): now also RN1.5 (R5.1); no longer RN1.6 (R6.1)
- net at JP12.1 (A), JP5.1 (A), JP7.2 (B): now also RN1.6 (R6.1); no longer RN1.7 (R7.1)
- net at JP10.1 (A), JP7.1 (A): now also RN1.7 (R7.1); no longer RN1.8 (R8.1)
- net at JP9.1 (A): now also RN1.10 (R7.2); no longer RN1.9 (R8.2)
- new net: C14.1, C15.1, C23.1, C24.1, R11.1, R12.1, R19.2, R20.1, U4.3 (HEATER+), U7.7 (V+)
- new net: Q1.1 (B), R25.2, U5.2 (VP)
- new net: C21.2, R15.1, RN1.16 (R1.2)
- new net: R22.1, U7.2 (-IN), U7.6 (OUT)
- new net: C20.2, U6.6 (OUT), U7.3 (+IN)
- new net: C16.1, C19.1, R20.2, U6.7 (V+)
- new net: J4.2 (Pin_2), Q1.2 (E), R25.1
- new net: J4.3 (Pin_3), Q1.3 (C), R26.1
- new net GNDREF: J4.4 (Pin_4), R26.2, U5.1 (VN)
Other:
- note added: "Temp sensor for resistor array"
- note removed: "Ref Zener Bias"
- title: ADR1399 refernce board -> ADR1399 reference board
- moved on the sheet: C1, C14, C15, C16, C17, C2, J3, JP1, JP10, JP11, JP12, JP2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
